Commit message: modify

File: baxter_bullet_env/models/baxter_description/urdf/baxter.urdf (robot description, URDF)
Before this commit: robot baxter, 57 links, 56 joints
Links:
- link head: geometry collision sphere radius=0.001; visual mesh filename=package://baxter_description/meshes/head/H0.DAE
- link l_gripper_l_finger_tip: geometry collision box size=0.016 0.007 0.037; visual mesh filename=package://rethink_ee_description/meshes/electric_gripper/fi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
- link l_gripper_r_finger_tip: geometry collision box size=0.016 0.007 0.037; visual mesh filename=package://rethink_ee_description/meshes/electric_gripper/fi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
- link left_lower_elbow: geometry collision cylinder length=0.10 radius=0.06; visual mesh filename=package://baxter_description/meshes/lower_elbow/E1.DAE
- link left_lower_forearm: geometry collision cylinder length=0.10 radius=0.06; visual mesh filename=package://baxter_description/meshes/lower_forearm/W1.DAE
- link left_lower_shoulder: geometry collision cylinder length=0.12 radius=0.06; visual mesh filename=package://baxter_description/meshes/lower_shoulder/S1.DAE
- link left_upper_elbow: geometry collision cylinder length=0.107 radius=0.06; visual mesh filename=package://baxter_description/meshes/upper_elbow/E0.DAE
- link left_upper_forearm: geometry collision cylinder length=0.088 radius=0.06; visual mesh filename=package://baxter_description/meshes/upper_forearm/W0.DAE
- link left_upper_shoulder: geometry collision cylinder length=0.2722 radius=0.06; visual mesh filename=package://baxter_description/meshes/upper_shoulder/S0.DAE
- link left_wrist: geometry collision cylinder length=0.165 radius=0.06; visual mesh filename=package://baxter_description/meshes/wrist/W2.DAE
- link pedestal: geometry collision mesh filename=package://baxter_description/meshes/base/pedestal_link_coll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; visual mesh filename=package://baxter_description/meshes/base/PEDESTAL.DAE
- link r_gripper_l_finger_tip: geometry collision box size=0.016 0.007 0.037; visual mesh filename=package://rethink_ee_description/meshes/electric_gripper/fi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
- link r_gripper_r_finger_tip: geometry collision box size=0.016 0.007 0.037; visual mesh filename=package://rethink_ee_description/meshes/electric_gripper/fi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
- link right_lower_elbow: geometry collision cylinder length=0.10 radius=0.06; visual mesh filename=package://baxter_description/meshes/lower_elbow/E1.DAE
- link right_lower_forearm: geometry collision cylinder length=0.10 radius=0.06; visual mesh filename=package://baxter_description/meshes/lower_forearm/W1.DAE
- link right_lower_shoulder: geometry collision cylinder length=0.12 radius=0.06; visual mesh filename=package://baxter_description/meshes/lower_shoulder/S1.DAE
- link right_upper_elbow: geometry collision cylinder length=0.107 radius=0.06; visual mesh filename=package://baxter_description/meshes/upper_elbow/E0.DAE
- link right_upper_forearm: geometry collision cylinder length=0.088 radius=0.06; visual mesh filename=package://baxter_description/meshes/upper_forearm/W0.DAE
- link right_upper_shoulder: geometry collision cylinder length=0.2722 radius=0.06; visual mesh filename=package://baxter_description/meshes/upper_shoulder/S0.DAE
- link right_wrist: geometry collision cylinder length=0.165 radius=0.06; visual mesh filename=package://baxter_description/meshes/wrist/W2.DAE
- link screen: geometry collision sphere radius=0.001; visual mesh filename=package://baxter_description/meshes/head/H1.DAE
- link torso: geometry collision mesh filename=package://baxter_description/meshes/torso/base_link_collisi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; visual mesh filename=package://baxter_description/meshes/torso/base_link.DAE
Joints:
- joint l_gripper_l_finger_joint: origin xyz=0.0 -0.0015 0.02 rpy=0 0 0 -> xyz=0.0 -0.0014999999999999996 0.02 rpy=0 0 0
- joint l_gripper_r_finger_joint: origin xyz=0.0 0.0015 0.02 rpy=0 0 0 -> xyz=0.0 0.0014999999999999996 0.02 rpy=0 0 0
- joint left_endpoint: origin xyz=0 0 0.1327 rpy=0 0 0 -> xyz=0 0 0.13269999999999998 rpy=0 0 0
- joint left_torso_arm_mount: origin xyz=0.0250508909425 0.219392814533 0.107748812049 rpy=-0.0074420066736 -0.00129546242287 0.78310045671 -> xyz=0.024645 0.219645 0.118588 rpy=0 0 0.7854
- joint r_gripper_l_finger_joint: origin xyz=0.0 -0.0015 0.02 rpy=0 0 0 -> xyz=0.0 -0.0014999999999999996 0.02 rpy=0 0 0
- joint r_gripper_r_finger_joint: origin xyz=0.0 0.0015 0.02 rpy=0 0 0 -> xyz=0.0 0.0014999999999999996 0.02 rpy=0 0 0
- joint right_endpoint: origin xyz=0 0 0.1327 rpy=0 0 0 -> xyz=0 0 0.13269999999999998 rpy=0 0 0
- joint right_torso_arm_mount: origin xyz=0.0248817669183 -0.220060922512 0.108693545459 rpy=0.000354590910292 0.00137984354452 -0.780560741676 -> xyz=0.024645 -0.219645 0.118588 rpy=0 0 -0.7854

Commit message: modify

File: baxter_bullet_env/models/baxter_description/urdf/baxter.urdf (robot description, URDF)
Before this commit: robot baxter, 57 links, 56 joints
Links:
- link l_gripper_l_finger_tip: geometry collision box size=0.042 0.0065 0.037; visual mesh filename=package://rethink_ee_description/meshes/electric_gripper/fi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
- link l_gripper_r_finger_tip: geometry collision box size=0.042 0.0065 0.037; visual mesh filename=package://rethink_ee_description/meshes/electric_gripper/fi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
- link r_gripper_l_finger_tip: geometry collision box size=0.042 0.0065 0.037; visual mesh filename=package://rethink_ee_description/meshes/electric_gripper/fi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
- link r_gripper_r_finger_tip: geometry collision box size=0.042 0.0065 0.037; visual mesh filename=package://rethink_ee_description/meshes/electric_gripper/fi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
